Commit message: Add meshes folder

File: urdf/widowx2.urdf (robot description, URDF)
Before this commit: robot widowx_arm, 11 links, 10 joints
Links:
- link base: geometry collision mesh filename=package://visual_servoing_powergrid/meshes/base_link.stl; visual mesh filename=package://visual_servoing_powergrid/meshes/base_link.stl
- link biceps_link: geometry collision mesh filename=package://visual_servoing_powergrid/meshes/biceps_link.stl; visual mesh filename=package://visual_servoing_powergrid/meshes/biceps_link.stl
- link forearm_link: geometry collision mesh filename=package://visual_servoing_powergrid/meshes/forearm_link.stl; visual mesh filename=package://visual_servoing_powergrid/meshes/forearm_link.stl
- link gripper_1_link: geometry collision mesh filename=package://visual_servoing_powergrid/meshes/gripper_hand_fix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; visual mesh filename=package://visual_servoing_powergrid/meshes/gripper_hand_fix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
- link gripper_2_link: geometry collision mesh filename=package://visual_servoing_powergrid/meshes/gripper_hand_fix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; visual mesh filename=package://visual_servoing_powergrid/meshes/gripper_hand_fix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
- link gripper_rail: geometry collision mesh filename=package://visual_servoing_powergrid/meshes/gripper_rail_lin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; visual mesh filename=package://visual_servoing_powergrid/meshes/gripper_rail_lin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
- link shoulder_link: geometry collision mesh filename=package://visual_servoing_powergrid/meshes/shoulder_link.stl; visual mesh filename=package://visual_servoing_powergrid/meshes/shoulder_link.stl
- link wrist_1_link: geometry collision mesh filename=package://visual_servoing_powergrid/meshes/wrist_1_link.stl; visual mesh filename=package://visual_servoing_powergrid/meshes/wrist_1_link.stl
- link wrist_2_link: geometry collision mesh filename=package://visual_servoing_powergrid/meshes/wrist_2_link.stl; visual mesh filename=package://visual_servoing_powergrid/meshes/wrist_2_link.stl
